Commit message: 在实际机器人上进行了测试，发现无线网不能满足需求

File: jaka_description/urdf/jaka.urdf.xacro (robot description, xacro)
@@ -223,5 +223,5 @@
     <joint name="joint_6" type="revolute">
         <axis xyz="0 0 1"/>
-        <limit effort="1000" lower="-3.14159265358" upper="3.14159265358" velocity="0.5"/>
+        <limit effort="1000" lower="${-3*pi/2.0}" upper="${3*pi/2.0}" velocity="0.5"/>
         <origin rpy="${-pi/2.0} 0 0" xyz="0 0.093 0"/>
         <parent link="link_5"/>

Commit message: 添加新版JAKAros驱动

File: jaka_description/urdf/jaka.urdf.xacro (robot description, xacro)
@@ -1,295 +1,209 @@
-<?xml version="1.0" ?>
-<robot name="jakaUr" xmlns:xacro="http://www.ros.org/wiki/xacro">
-    <xacro:property name="pi" value="3.14159265358"/>
-    <material name="blue">
-        <color rgba="0 0 0.8 1"/>
-    </material>
-    <material name="black">
-        <color rgba="0 0 0 1"/>
-    </material>
-    <material name="white">
-        <color rgba="1 1 1 1"/>
-    </material>
-    <!--############## link ##############-->
-    <link name="world"/>
-    <link name="bottom_link">
-        <!--visual><origin xyz=" 0 0 -0.04"  rpy="0 0 0"/><geometry><box size="1 1 0.02" /></geometry><material name="Brown" /></visual><collision><origin xyz=" 0 0 -0.04"  rpy="0 0 0"/><geometry><box size="1 1 0.02" /></geometry></collision>-->
-        <inertial>
-            <mass value="5"/>
-            <inertia ixx="0.2" ixy="0.0" ixz="0.0" iyy="0.2" iyz="0.0" izz="0.1"/>
-        </inertial>
-    </link>
-    <link name="base_link">
-        <visual>
-            <!--origin rpy="0 ${pi / 2} 0" xyz="0 0 0.0198"/>-->
-            <origin rpy="0 0 0" xyz="0 0 -0.0005"/>
-            <geometry>
-                <mesh filename="package://jaka_description/meshes/p11.dae"/>
-            </geometry>
-            <material name="white">
-                <color rgba="1 1 1 1"/>
-            </material>
-        </visual>
-        <collision>
-            <geometry>
-                <mesh filename="package://jaka_description/meshes/p11.dae"/>
-            </geometry>
-            <origin rpy="0 0 0" xyz="0 0 -0.0005"/>
-        </collision>
-        <!--inertial><mass value="5"/><inertia ixx="0.2" ixy="0.0" ixz="0.0" iyy="0.2" iyz="0.0" izz="0.1"/></inertial-->
-    </link>
-    <link name="link_1">
-        <visual>
-            <geometry>
-                <mesh filename="package://jaka_description/meshes/p22.dae"/>
-            </geometry>
-            <material name="white">
-                <color rgba="1 1 1 1"/>
-            </material>
-            <!--origin rpy=" ${pi/2.0}  0  ${pi/2.0}" xyz="0 0 0"/>-->
-            <origin rpy=" 0  0  0" xyz="0 0 0"/>
-        </visual>
-        <collision>
-            <geometry>
-                <mesh filename="package://jaka_description/meshes/p22.dae"/>
-            </geometry>
-            <origin rpy=" 0  0  0" xyz="0 0 0"/>
-        </collision>
-        <inertial>
-            <mass value="8"/>
-            <inertia ixx="0.3" ixy="0.0" ixz="0.0" iyy="0.3" iyz="0.0" izz="0.2"/>
-        </inertial>
-    </link>
-    <link name="link_2">
-        <visual>
-            <geometry>
-                <mesh filename="package://jaka_description/meshes/p35.dae"/>
-            </geometry>
-            <!--origin rpy="${pi/2.0}  ${pi} ${pi/2.0}" xyz="-0.1595 0 -0.115"/>-->
-            <material name="white">
-                <color rgba="1 1 1 1"/>
-            </material>
-            <origin rpy="${pi/2.0} ${pi} ${pi/2.0}" xyz="0 0 0.005 "/>
-            <material name="white">
-                <color rgba="1 1 1 1"/>
-            </material>
-        </visual>
-        <collision>
-            <geometry>
-                <mesh filename="package://jaka_description/meshes/p35.dae"/>
-            </geometry>
-            <origin rpy="${pi/2.0} ${pi} ${pi/2.0}" xyz="0 0 0.005 "/>
-        </collision>
-        <inertial>
-            <mass value="6"/>
-            <inertia ixx="0.25" ixy="0.0" ixz="0.0" iyy="0.25" iyz="0.0" izz="0.15"/>
-        </inertial>
-    </link>
-    <link name="link_3">
-        <visual>
-            <geometry>
-                <mesh filename="package://jaka_description/meshes/p44.dae"/>
-            </geometry>
-            <material name="white">
-                <color rgba="1 1 1 1"/>
-            </material>
-            <origin rpy="${-pi/2.0} 0 ${-pi/2.0}" xyz="0.303 0 -0.013"/>
-        </visual>
-        <collision>
-            <geometry>
-                <mesh filename="package://jaka_description/meshes/p44.dae"/>
-            </geometry>
-            <origin rpy="${-pi/2.0} 0 ${-pi/2.0}" xyz="0.303 0 -0.013"/>
-        </collision>
-        <inertial>
-            <mass value="8"/>
-            <inertia ixx="0.3" ixy="0.0" ixz="0.0" iyy="0.3" iyz="0.0" izz="0.2"/>
-        </inertial>
-    </link>
-    <link name="link_4">
-        <visual>
-            <geometry>
-                <mesh filename="package://jaka_description/meshes/p55.dae"/>
-            </geometry>
-            <origin rpy="${pi/2.0} 0 ${pi/2.0}" xyz="0.00 0 0.00"/>
-            <material name="white">
-                <color rgba="1 1 1 1"/>
-            </material>
-        </visual>
-        <collision>
-            <geometry>
-                <mesh filename="package://jaka_description/meshes/p55.dae"/>
-            </geometry>
-            <origin rpy="${pi/2.0} 0 ${pi/2.0}" xyz="0.00 0 0.00"/>
-        </collision>
-        <inertial>
-            <mass value="5"/>
-            <inertia ixx="0.2" ixy="0.0" ixz="0.0" iyy="0.2" iyz="0.0" izz="0.15"/>
-        </inertial>
-    </link>
-    <link name="link_5">
-        <visual>
-            <geometry>
-                <mesh filename="package://jaka_description/meshes/p66.dae"/>
-            </geometry>
-            <origin rpy="${pi} 0 ${-pi/2.0}" xyz="0 0 0"/>
-            <material name="white">
-                <color rgba="1 1 1 1"/>
-            </material>
-        </visual>
-        <collision>
-            <geometry>
-                <mesh filename="package://jaka_description/meshes/p66.dae"/>
-            </geometry>
-            <origin rpy="${pi} 0 ${-pi/2.0}" xyz="0 0 0"/>
-        </collision>
-        <inertial>
-            <mass value="4"/>
-            <inertia ixx="0.1" ixy="0.0" ixz="0.0" iyy="0.1" iyz="0.0" izz="0.07"/>
-        </inertial>
-    </link>
-    <link name="link_6">
-        <visual>
-            <geometry>
-                <mesh filename="package://jaka_description/meshes/p77.dae"/>
-            </geometry>
-            <origin rpy="0 ${-pi/2.0}  0" xyz="0 0 -0.0335"/>
-        </visual>
-        <collision>
-            <geometry>
-                <mesh filename="package://jaka_description/meshes/p77.dae"/>
-            </geometry>
-            <origin rpy="0 ${-pi/2.0}  0" xyz="0 0 -0.0335"/>
-        </collision>
-        <inertial>
-            <mass value="2"/>
-            <inertia ixx="0.07" ixy="0.0" ixz="0.0" iyy="0.07" iyz="0.0" izz="0.04"/>
-        </inertial>
-    </link>
-    <link name="ee_link">
-        <collision>
-            <geometry>
-                <box size="0.01 0.01 0.01"/>
-            </geometry>
-            <origin rpy="0 0 0" xyz="-0.01 0 0"/>
-        </collision>
-    </link>
-    <!--############## joint ##############-->
-    <joint name="world_joint" type="fixed">
-        <origin rpy="0 0 0" xyz="0 0 0"/>
-        <parent link="world"/>
-        <child link="base_link"/>
-    </joint>
-    <joint name="bottom_joint" type="fixed">
-        <origin rpy="0 0 0" xyz="0 0 0"/>
-        <parent link="base_link"/>
-        <child link="bottom_link"/>
-    </joint>
-    <joint name="joint_1" type="revolute">
-        <axis xyz="0 0 1"/>
-        <limit effort="1000" lower="-3.14159265358" upper="3.14159265358" velocity="0.5"/>
-        <origin rpy="0 0 0" xyz="0 0 0.114"/>
-        <parent link="base_link"/>
-        <child link="link_1"/>
-    </joint>
-    <joint name="joint_2" type="revolute">
-        <axis xyz="0 0 1"/>
-        <limit effort="1000" lower="-1.58" upper="4.71238898" velocity="0.5"/>
-        <origin rpy="${pi/2.0} 0 0" xyz="0 0 0"/>
-        <parent link="link_1"/>
-        <child link="link_2"/>
-    </joint>
-    <joint name="joint_3" type="revolute">
-        <axis xyz="0 0 1"/>
-        <limit effort="1000" lower="-3.14159265358" upper="3.14159265358" velocity="0.5"/>
-        <origin rpy="0 0 0" xyz="0.353 0 0"/>
-        <parent link="link_2"/>
-        <child link="link_3"/>
-    </joint>
-    <joint name="joint_4" type="revolute">
-        <axis xyz="0 0 1"/>
-        <limit effort="1000" lower="-3.14159265358" upper="3.14159265358" velocity="0.5"/>
-        <origin rpy="0 0 0" xyz="0.303 0 -0.1155"/>
-        <parent link="link_3"/>
-        <child link="link_4"/>
-    </joint>
-    <joint name="joint_5" type="revolute">
-        <axis xyz="0 0 1"/>
-        <limit effort="1000" lower="-3.14159265358" upper="3.14159265358" velocity="0.5"/>
-        <origin rpy="${pi/2.0} 0 0" xyz="0 -0.1025 0"/>
-        <parent link="link_4"/>
-        <child link="link_5"/>
-    </joint>
-    <joint name="joint_6" type="revolute">
-        <axis xyz="0 0 1"/>
-        <limit effort="1000" lower="${-3*pi/2.0}" upper="${3*pi/2.0}" velocity="0.5"/>
-        <origin rpy="${-pi/2.0} 0 0" xyz="0 0.093 0"/>
-        <parent link="link_5"/>
-        <child link="link_6"/>
-    </joint>
-    <joint name="ee_fixed_joint" type="fixed">
-        <parent link="link_6" />
-        <child link = "ee_link" />
-        <origin xyz="0.0 0.0 0.0" rpy="0.0 0.0 0.0" />
-    </joint>
-    <transmission name="joint_1_trans">
-        <type>transmission_interface/SimpleTransmission</type>
-        <actuator name="$joint_1_motor">
-            <mechanicalReduction>1</mechanicalReduction>
-        </actuator>
-        <joint name="joint_1">
-            <hardwareInterface>PositionJointInterface</hardwareInterface>
-        </joint>
-    </transmission>
-    <transmission name="joint_2_trans">
-        <type>transmission_interface/SimpleTransmission</type>
-        <actuator name="$joint_2_motor">
-            <mechanicalReduction>1</mechanicalReduction>
-        </actuator>
-        <joint name="joint_2">
-            <hardwareInterface>PositionJointInterface</hardwareInterface>
-        </joint>
-    </transmission>
-    <transmission name="joint_3_trans">
-        <type>transmission_interface/SimpleTransmission</type>
-        <actuator name="joint_3_motor">
-            <mechanicalReduction>1</mechanicalReduction>
-        </actuator>
-        <joint name="joint_3">
-            <hardwareInterface>PositionJointInterface</hardwareInterface>
-        </joint>
-    </transmission>
-    <transmission name="joint_4_trans">
-        <type>transmission_interface/SimpleTransmission</type>
-        <actuator name="joint_4_motor">
-            <mechanicalReduction>1</mechanicalReduction>
-        </actuator>
-        <joint name="joint_4">
-            <hardwareInterface>PositionJointInterface</hardwareInterface>
-        </joint>
-    </transmission>
-    <transmission name="joint_5_trans">
-        <type>transmission_interface/SimpleTransmission</type>
-        <actuator name="joint_5_motor">
-            <mechanicalReduction>1</mechanicalReduction>
-        </actuator>
-        <joint name="joint_5">
-            <hardwareInterface>PositionJointInterface</hardwareInterface>
-        </joint>
-    </transmission>
-    <transmission name="joint_6_trans">
-        <type>transmission_interface/SimpleTransmission</type>
-        <actuator name="joint_6_motor">
-            <mechanicalReduction>1</mechanicalReduction>
-        </actuator>
-        <joint name="joint_6">
-            <hardwareInterface>PositionJointInterface</hardwareInterface>
-        </joint>
-    </transmission>
-    <!--########### ros_control plugin ###########-->
-    <gazebo>
-        <plugin filename="libgazebo_ros_control.so" name="gazebo_ros_control">
-            <robotNamespace>/jakaUr</robotNamespace>
-        </plugin>
-    </gazebo>
+<?xml version="1.0" encoding="utf-8"?>
+<!-- This URDF was automatically created by SolidWorks to URDF Exporter! Originally created by Stephen Brawner (brawner@gmail.com)
+     Commit Version: 1.5.1-0-g916b5db  Build Version: 1.5.7152.31018
+     For more information, please see http://wiki.ros.org/sw_urdf_exporter -->
+<robot name="jaka_description">
+  <link name="world"/>
+  <link name="base_link">
+    <inertial>
+      <origin xyz="0.0078045 0.02052 0.0017471" rpy="0 0 0" />
+      <mass value="0.51461" />
+      <inertia ixx="0.00062136" ixy="3.2169E-06" ixz="-3.6994E-09" iyy="0.0013529" iyz="1.2577E-10" izz="0.00086645" />
+    </inertial>
+    <visual>
+      <origin xyz="0 0 0" rpy="0 0 0" />
+      <geometry>
+        <mesh filename="package://jaka_description/meshes/base_link.STL" />
+      </geometry>
+      <material name="">
+        <color rgba="1 1 1 1" />
+      </material>
+    </visual>
+    <collision>
+      <origin xyz="0 0 0" rpy="0 0 0" />
+      <geometry>
+        <mesh filename="package://jaka_description/meshes/base_link.STL" />
+      </geometry>
+    </collision>
+  </link>
+  <joint name="fixed_joint" type="fixed">
+    <origin xyz="0 0 0" rpy="0 0 0" />
+    <parent link="world" />
+    <child link="base_link" />
+  </joint>
+  <link name="link1">
+    <inertial>
+      <origin xyz="0.0033217 0.078637 -9.9561E-07" rpy="0 0 0" />
+      <mass value="1.9281" />
+      <inertia ixx="0.0054895" ixy="1.9288E-06" ixz="-8.0735E-09" iyy="0.0038887" iyz="-1.0336E-08" izz="0.0056434" />
+    </inertial>
+    <visual>
+      <origin xyz="0 0 0" rpy="0 0 0" />
+      <geometry>
+        <mesh filename="package://jaka_description/meshes/link1.STL" />
+      </geometry>
+      <material name="">
+        <color rgba="1 1 1 1" />
+      </material>
+    </visual>
+    <collision>
+      <origin xyz="0 0 0" rpy="0 0 0" />
+      <geometry>
+        <mesh filename="package://jaka_description/meshes/link1.STL" />
+      </geometry>
+    </collision>
+  </link>
+  <joint name="joint1" type="continuous">
+    <origin xyz="0.0068395 -0.0017473 0.040967" rpy="1.5708 0 1.5708" />
+    <parent link="base_link" />
+    <child link="link1" />
+    <axis xyz="0 1 0" />
+  </joint>
+  <link name="link2">
+    <inertial>
+      <origin xyz="0.180000209977346 0.0790053241117423 1.81612678296084E-06" rpy="0 0 0" />
+      <mass value="5.46194601044026" />
+      <inertia ixx="0.012915357360266" ixy="-3.31771617532355E-08" ixz="-9.02794658605086E-09" iyy="0.0177711235371075" iyz="-2.29869349851466E-09" izz="0.0212789850441894" />
+    </inertial>
+    <visual>
+      <origin xyz="0 0 0" rpy="0 0 0" />
+      <geometry>
+        <mesh filename="package://jaka_description/meshes/link2.STL" />
+      </geometry>
+      <material name="">
+        <color rgba="1 1 1 1" />
+      </material>
+    </visual>
+    <collision>
+      <origin xyz="0 0 0" rpy="0 0 0" />
+      <geometry>
+        <mesh filename="package://jaka_description/meshes/link2.STL" />
+      </geometry>
+    </collision>
+  </link>
+  <joint name="joint2" type="continuous">
+    <origin xyz="0.06407 0.08015 0" rpy="-3.1416 -1.5708 1.5708" />
+    <!-- rpy="-3.1416 0.61321 1.5708"-->
+    <parent link="link1" />
+    <child link="link2" />
+    <axis xyz="0 -1 0" />
+  </joint>
+  <link name="link3">
+    <inertial>
+      <origin xyz="0.154631179365296 0.051491742581724 -9.87671775865007E-07" rpy="0 0 0" />
+      <mass value="2.10990539238288" />
+      <inertia ixx="0.002372120404392" ixy="-0.00148686871157693" ixz="1.61083887908488E-07" iyy="0.0128780808874665" iyz="1.06256446469924E-09" izz="0.0132375017255301" />
+    </inertial>
+    <visual>
+      <origin xyz="0 0 0" rpy="0 0 0" />
+      <geometry>
+        <mesh filename="package://jaka_description/meshes/link3.STL" />
+      </geometry>
+      <material name="">
+        <color rgba="1 1 1 1" />
+      </material>
+    </visual>
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
File: jaka_description/urdf/jaka_description.urdf (robot description, URDF)
Before this commit: robot jakaUr, 10 links, 9 joints
Links:
- removed link bottom_link
- removed link ee_link
- removed link link_1
- removed link link_2
- removed link link_3
- removed link link_4
- removed link link_5
- removed link link_6
- removed link world
- added link link1, mass 1.9281; collision mesh filename=package://jaka_description/meshes/link1.STL; visual mesh filename=package://jaka_description/meshes/link1.STL
- added link link2, mass 5.46194601044026; collision mesh filename=package://jaka_description/meshes/link2.STL; visual mesh filename=package://jaka_description/meshes/link2.STL
- added link link3, mass 2.10990539238288; collision mesh filename=package://jaka_description/meshes/link3.STL; visual mesh filename=package://jaka_description/meshes/link3.STL
- added link link4, mass 0.707388000054209; collision mesh filename=package://jaka_description/meshes/link4.STL; visual mesh filename=package://jaka_description/meshes/link4.STL
- added link link5, mass 0.806925581335565; collision mesh filename=package://jaka_description/meshes/link5.STL; visual mesh filename=package://jaka_description/meshes/link5.STL
- added link link6, mass 0.180494526010387; collision mesh filename=package://jaka_description/meshes/link6.STL; visual mesh filename=package://jaka_description/meshes/link6.STL
- link base_link: mass None -> 0.51461; geometry collision mesh filename=package://jaka_description/meshes/base_link.STL; visual mesh filename=package://jaka_description/meshes/base_link.STL
Joints:
- removed joint bottom_joint
- removed joint ee_fixed_joint
- removed joint joint_1
- removed joint joint_2
- removed joint joint_3
- removed joint joint_4
- removed joint joint_5
- removed joint joint_6
- removed joint world_joint
- added joint joint1: type continuous, parent base_link, child link1, origin xyz=0.0068395 -0.0017473 0.040967 rpy=1.5708 0 1.5708, axis 0 1 0
- added joint joint2: type continuous, parent link1, child link2, origin xyz=0.06407 0.08015 0 rpy=-3.1416 -1.5708 1.5708, axis 0 -1 0
- added joint joint3: type continuous, parent link2, child link3, origin xyz=0.36 0 0 rpy=0 3.1415926 -3.1415926, axis 0 1 0
- added joint joint4: type continuous, parent link3, child link4, origin xyz=0.303 -0.0054826 0 rpy=-1.5708 0 -1.5708, axis -1 0 0
- added joint joint5: type continuous, parent link4, child link5, origin xyz=0.04546 -0.067529 0 rpy=3.1415926 0 1.5708, axis -1 0 0
- added joint joint6: type continuous, parent link5, child link6, origin xyz=-0.045971 -0.069408 0 rpy=0 -1.5708 0, axis 0 -1 0
